Commit message: Fix teleop mapping, point cloud frame and braking skid; add IR line array
Teleop
- add a generic HID gamepad mapping (SHANWAN, 8BitDo, Xbox over Bluetooth)
- command topics use a queue of 1, joystick repeat raised to 30 Hz

Simulation
- build the point cloud from the depth image so it is in the optical frame
- limit braking in the diff drive plugin, which stops the robot skidding
  and yawing on every stop; angular limit raised to 8 rad/s2
- 8 channel analog IR line sensor array on /ir/analog (0 to 5 V) and a
  line world to test it on
- gripper jaw mass and inertia recomputed for PLA at 1240 kg/m3
- depth camera resolution and rate are xacro properties, set to
  1920 x 1080 at 60 Hz
- maze physics step 2 ms, helper nodes no longer follow /clock

Docker
- add depth_image_proc to the image and an init process to the service

Co-authored-by: podalanga <145194987+podalanga@users.noreply.github.com>

File: src/trident_description/urdf/trident.gazebo.xacro (robot description, xacro)
@@ -30,6 +30,8 @@
       <wheel_separation>${2*wheel_y}</wheel_separation>
       <wheel_radius>${wheel_radius}</wheel_radius>
-      <max_linear_acceleration>1.0</max_linear_acceleration>
-      <max_angular_acceleration>4.0</max_angular_acceleration>
+      <max_linear_acceleration>${drive_accel_linear}</max_linear_acceleration>
+      <min_linear_acceleration>${-drive_accel_linear}</min_linear_acceleration>
+      <max_angular_acceleration>${drive_accel_angular}</max_angular_acceleration>
+      <min_angular_acceleration>${-drive_accel_angular}</min_angular_acceleration>
       <topic>cmd_vel</topic>
       <odom_topic>odom</odom_topic>
@@ -70,10 +72,12 @@
   </gazebo>
   <!-- == D435: RGB-D sensor on the depth origin, looking along +X.
-       Depth FOV 87 deg x 58 deg at 848 x 480. Near clip 0.1 m keeps the holder lip out of view.
-       Messages are stamped with the optical frame so point clouds line up in RViz. == -->
+       Depth FOV 87 deg x 58 deg. Near clip 0.1 m keeps the holder lip out of view.
+       Images are stamped with the optical frame. Gazebo's own point cloud is not used: it has
+       X forward but carries the same optical frame id, so the cloud is built in ROS from the
+       depth image instead (see trident_gazebo sim.launch.py). == -->
   <gazebo reference="camera_depth_frame">
     <sensor name="d435" type="rgbd_camera">
       <always_on>true</always_on>
-      <update_rate>30</update_rate>
+      <update_rate>${d435_rate}</update_rate>
       <visualize>false</visualize>
       <topic>camera</topic>
@@ -82,6 +86,6 @@
         <horizontal_fov>1.5184</horizontal_fov>
         <image>
-          <width>848</width>
-          <height>480</height>
+          <width>${d435_width}</width>
+          <height>${d435_height}</height>
           <format>R8G8B8</format>
         </image>
@@ -104,3 +108,39 @@
     </sensor>
   </gazebo>
+  <!-- == IR line sensor array: one tiny camera per channel, looking straight down.
+       ir_sensor_frame has +X toward the floor, Y across the board, Z toward the front.
+       trident_gazebo/scripts/ir_array.py turns the images into one analog reading per channel. == -->
+  <xacro:macro name="ir_channel" params="index">
+    <gazebo reference="ir_sensor_frame">
+      <sensor name="ir_ch${index}" type="camera">
+        <!-- 1 mm below the board face, offset along the row -->
+        <pose>0.001 ${ir_center_y + (index - (ir_channels - 1) / 2.0) * ir_pitch} ${ir_center_x} 0 0 0</pose>
+        <always_on>true</always_on>
+        <update_rate>${ir_rate}</update_rate>
+        <visualize>false</visualize>
+        <topic>ir/ch${index}</topic>
+        <camera>
+          <!-- about an 8 mm spot on the floor from 7 mm up, like a reflectance sensor -->
+          <horizontal_fov>1.0</horizontal_fov>
+          <image>
+            <width>8</width>
+            <height>8</height>
+            <format>R8G8B8</format>
+          </image>
+          <clip>
+            <near>0.002</near>
+            <far>0.1</far>
+          </clip>
+        </camera>
+      </sensor>
+    </gazebo>
+  </xacro:macro>
+  <!-- xacro has no for loop, so the macro calls itself until the last channel -->
+  <xacro:macro name="ir_array" params="index:=0">
+    <xacro:if value="${index &lt; ir_channels}">
+      <xacro:ir_channel index="${index}"/>
+      <xacro:ir_array index="${index + 1}"/>
+    </xacro:if>
+  </xacro:macro>
+  <xacro:ir_array/>
 </robot>

File: src/trident_description/urdf/trident.urdf.xacro (robot description, xacro)
@@ -24,4 +24,8 @@
   <xacro:property name="wheel_effort"     value="0.05"/>      <!-- N m, stall torque at the wheel -->
   <xacro:property name="wheel_velocity"   value="31.4"/>      <!-- rad/s, no-load speed (300 rpm) -->
+  <!-- Acceleration limits for the diff drive, applied to speeding up and to braking.
+       Without the braking limit the wheels stop dead and the robot skids and yaws. -->
+  <xacro:property name="drive_accel_linear"  value="1.0"/>    <!-- m/s^2 -->
+  <xacro:property name="drive_accel_angular" value="8.0"/>    <!-- rad/s^2 -->
   <!-- Caster: dome radius 10.5 mm, centre at castor_wheel_sphere_coords.
        In CAD the dome bottom sits 0.74 mm above the wheel contact plane. The collision radius
@@ -45,4 +49,16 @@
   <xacro:property name="d435_depth_x"     value="${d435_len_x - 0.0042}"/>
   <xacro:property name="d435_depth_y"     value="${d435_center_y + 0.0175}"/>
+  <!-- Simulated stream. 1920 x 1080 at 60 Hz is beyond what a real D435 does (depth tops out at
+       1280 x 720, 30 Hz) and is heavy to render. Lower these three first if the sim runs slow,
+       for example 424 x 240 at 15 Hz. -->
+  <xacro:property name="d435_width"       value="1920"/>
+  <xacro:property name="d435_height"      value="1080"/>
+  <xacro:property name="d435_rate"        value="60"/>
+  <!-- IR line sensor array: channels sit in a row across the board (along Y) -->
+  <xacro:property name="ir_channels"      value="8"/>
+  <xacro:property name="ir_pitch"         value="0.015"/>     <!-- m, centre to centre -->
+  <xacro:property name="ir_center_y"      value="0.0007"/>    <!-- board centre in ir_base_link -->
+  <xacro:property name="ir_center_x"      value="-0.008"/>
+  <xacro:property name="ir_rate"          value="20"/>        <!-- Hz -->
   <!-- ============================ base ============================ -->
   <link name="base_footprint"/>
@@ -133,7 +149,8 @@
   <link name="gripper_drive_link">
     <inertial>
-      <origin xyz="0.037012 0.035574 0" rpy="0 0 0"/>
-      <mass value="0.029369"/>
-      <inertia ixx="3.2335E-06" ixy="3.1111E-06" ixz="0" iyy="2.6949E-05" iyz="0" izz="2.987E-05"/>
+      <!-- PLA, 1240 kg/m3, computed from the mesh (11.81 cm3) -->
+      <origin xyz="0.03072 -0.01303 0" rpy="0 0 0"/>
+      <mass value="0.014648"/>
+      <inertia ixx="1.7643E-06" ixy="2.1546E-06" ixz="0" iyy="1.3239E-05" iyz="0" izz="1.4847E-05"/>
     </inertial>
     <visual>
@@ -158,7 +175,8 @@
     <inertial>
       <origin xyz="0.0233005821511302 0.00658223410359155 -0.00252490161223871" rpy="0 0 0"/>
-      <mass value="0.0210562573264184"/>
-      <inertia ixx="2.44538134970393E-06" ixy="-1.90484190620614E-06" ixz="1.21407959125207E-06"
-               iyy="1.91707326281041E-05" iyz="3.43006008331818E-07" izz="2.06767405330995E-05"/>
+      <!-- PLA, 1240 kg/m3, computed from the mesh (16.29 cm3) -->
+      <mass value="0.020201"/>
+      <inertia ixx="2.3362E-06" ixy="-1.8337E-06" ixz="1.1640E-06"
+               iyy="1.8337E-05" iyz="3.2888E-07" izz="1.9772E-05"/>
     </inertial>
     <visual>

Commit message: Add mission arena world, IMU and split odometry bridge
Simulation
- arena world (xacro): curved entry line, start square, three T-marked pick
  bays with coins, three drop squares, QR placards and textured walls
- pick_order, drop_order and obstacles launch arguments shuffle a run
- IMU on the chassis with gyro and accelerometer noise
- bridge config split: common topics, raw Gazebo odometry, EKF inputs
- optional Gaussian noise on the IR array readings
- make_textures.py regenerates the QR codes and wall panels

Docker
- robot_localization, RTAB-Map, Nav2, zbar_ros and python3-qrcode

Co-authored-by: podalanga <145194987+podalanga@users.noreply.github.com>

File: src/trident_description/urdf/trident.gazebo.xacro (robot description, xacro)
@@ -108,4 +108,26 @@
     </sensor>
   </gazebo>
+  <!-- == IMU: needs the Imu system plugin in the world (see arena.sdf.xacro).
+       Worlds without it simply get no /imu topic. == -->
+  <gazebo reference="imu_link">
+    <sensor name="imu" type="imu">
+      <always_on>true</always_on>
+      <update_rate>${imu_rate}</update_rate>
+      <topic>imu</topic>
+      <ignition_frame_id>imu_link</ignition_frame_id>
+      <imu>
+        <angular_velocity>
+            <x><noise type="gaussian"><mean>0</mean><stddev>${imu_gyro_noise}</stddev></noise></x>
+            <y><noise type="gaussian"><mean>0</mean><stddev>${imu_gyro_noise}</stddev></noise></y>
+            <z><noise type="gaussian"><mean>0</mean><stddev>${imu_gyro_noise}</stddev></noise></z>
+        </angular_velocity>
+        <linear_acceleration>
+            <x><noise type="gaussian"><mean>0</mean><stddev>${imu_accel_noise}</stddev></noise></x>
+            <y><noise type="gaussian"><mean>0</mean><stddev>${imu_accel_noise}</stddev></noise></y>
+            <z><noise type="gaussian"><mean>0</mean><stddev>${imu_accel_noise}</stddev></noise></z>
+        </linear_acceleration>
+      </imu>
+    </sensor>
+  </gazebo>
   <!-- == IR line sensor array: one tiny camera per channel, looking straight down.
        ir_sensor_frame has +X toward the floor, Y across the board, Z toward the front.

File: src/trident_description/urdf/trident.urdf.xacro (robot description, xacro)
@@ -61,4 +61,9 @@
   <xacro:property name="ir_center_x"      value="-0.008"/>
   <xacro:property name="ir_rate"          value="20"/>        <!-- Hz -->
+  <!-- IMU (MPU6050 class) flat on the chassis plate between the wheels -->
+  <xacro:property name="imu_xyz"          value="0.03 0 0.012"/>
+  <xacro:property name="imu_rate"         value="100"/>       <!-- Hz -->
+  <xacro:property name="imu_gyro_noise"   value="0.002"/>     <!-- rad/s, standard deviation -->
+  <xacro:property name="imu_accel_noise"  value="0.02"/>      <!-- m/s^2, standard deviation -->
   <!-- ============================ base ============================ -->
   <link name="base_footprint"/>
@@ -293,4 +298,12 @@
     <origin xyz="0 0 0" rpy="0 ${PI/2} 0"/>
   </joint>
+  <!-- ============================ IMU ============================ -->
+  <!-- Frame only, the board weighs next to nothing. Axes match base_link. -->
+  <link name="imu_link"/>
+  <joint name="imu_joint" type="fixed">
+    <parent link="base_link"/>
+    <child link="imu_link"/>
+    <origin xyz="${imu_xyz}" rpy="0 0 0"/>
+  </joint>
   <!-- Gazebo-only tags (friction, plugins, sensors) -->
   <xacro:include filename="$(find trident_description)/urdf/trident.gazebo.xacro"/>
